Commit message: added controllers

File: urdf/arm_meshed.urdf (robot description, URDF)
Before this commit: robot arm_mesh, 8 links, 7 joints
Links:
- link base: mass 0.120 -> 0.170
- link claw_L: geometry collision mesh filename=package://robotic_arm_pkg/meshes/gripper_claw_L.stl scale=0.001 0.001 0.001; visual mesh filename=package://robotic_arm_pkg/meshes/gripper_claw_L.stl scale=0.001 0.001 0.001
- link claw_R: geometry collision mesh filename=package://robotic_arm_pkg/meshes/gripper_claw_R.stl scale=0.001 0.001 0.001; visual mesh filename=package://robotic_arm_pkg/meshes/gripper_claw_R.stl scale=0.001 0.001 0.001
- link gripper_base: geometry collision mesh filename=package://robotic_arm_pkg/meshes/gripper_base.stl scale=0.001 0.001 0.001; visual mesh filename=package://robotic_arm_pkg/meshes/gripper_base.stl scale=0.001 0.001 0.001
- link link2: geometry collision box size=0.025 0.054 0.12; visual mesh filename=package://robotic_arm_pkg/meshes/link2.stl scale=0.001 0.001 0.001
- link link3: geometry collision box size=0.03 0.04 0.14; visual mesh filename=package://robotic_arm_pkg/meshes/link3.stl scale=0.001 0.001 0.001
- link link4: geometry collision mesh filename=package://robotic_arm_pkg/meshes/link4.stl scale=0.001 0.001 0.001; visual mesh filename=package://robotic_arm_pkg/meshes/link4.stl scale=0.001 0.001 0.001
