Commit message: initial commit

File: robotic_arm_pkg/urdf/arm_meshed.urdf (robot description, URDF)
Before this commit: robot arm_mesh, 8 links, 7 joints
Joints:
- joint base_link1: limit lower=-3.14 upper=3.14 effort=1000.0 velocity=0.5 -> lower=-1.57 upper=1.57 effort=1000.0 velocity=0.5

Commit message: modified urdf and mesh files

File: robotic_arm_pkg/urdf/arm_meshed.urdf (robot description, URDF)
Before this commit: robot arm_mesh, 8 links, 7 joints
Links:
- removed link link3
- added link link3bot; collision box size=0.03 0.035 0.08; visual mesh filename=package://robotic_arm_pkg/meshes/link3bot.stl scale=0.001 0.001 0.001
- added link link3top; collision box size=0.03 0.035 0.055; visual mesh filename=package://robotic_arm_pkg/meshes/link3top.stl scale=0.001 0.001 0.001
- link base: mass 0.170 -> None; geometry collision mesh filename=package://robotic_arm_pkg/meshes/base.stl scale=0.001 0.001 0.001; visual mesh filename=package://robotic_arm_pkg/meshes/base.stl scale=0.001 0.001 0.001
- link gripper_base: mass 0.020 -> None
- link link1: mass 0.075 -> None; geometry collision mesh filename=package://robotic_arm_pkg/meshes/link1.stl scale=0.001 0.001 0.001; visual mesh filename=package://robotic_arm_pkg/meshes/link1.stl scale=0.001 0.001 0.001
- link link2: mass 0.018 -> None; geometry collision box size=0.025 0.054 0.116; visual mesh filename=package://robotic_arm_pkg/meshes/link2.stl scale=0.001 0.001 0.001
- link link4: mass 0.025 -> None
Joints:
- removed joint link2_link3
- removed joint link3_link4
- added joint link2_link3bot: type revolute, parent link2, child link3bot, origin xyz=0 0 0.095 rpy=0 0 0, axis 0 1 0, limit lower=-1.57 upper=1.57 effort=1000.0 velocity=0.5
- added joint link3bot_link3top: type revolute, parent link3bot, child link3top, origin xyz=0 0 0.045 rpy=0 0 0, axis 0 0 1, limit lower=-1.57 upper=1.57 effort=1000.0 velocity=0.5
- added joint link3top_link4: type revolute, parent link3top, child link4, origin xyz=0 0 0.04 rpy=0 0 0, axis 0 1 0, limit lower=-1.57 upper=1.57 effort=1000.0 velocity=0.5
- joint base_link1: origin xyz=0 0 0.0175 rpy=0 0 0 -> xyz=0 0 0.033 rpy=0 0 0
- joint gripper_base_claw_L: origin xyz=0 -0.0125 0.01 rpy=0 0 0 -> xyz=0 -0.008 0.018 rpy=0 0 0
- joint gripper_base_claw_R: origin xyz=0 0.0035 0.012 rpy=0 0 0 -> xyz=0 0.008 0.018 rpy=0 0 0
- joint link1_link2: origin xyz=0 0 0.042 rpy=0 0 0 -> xyz=0 0 0.05 rpy=0 0 0
- joint link4_gripper_base: origin xyz=-0.01 0 0.06 rpy=0 0 0 -> xyz=-0.01 0 0.055 rpy=0 0 0

File: robotic_arm_pkg/urdf/original_urdf/arm_meshed.urdf (robot description, URDF)
Before this commit: robot arm_mesh, 9 links, 8 joints
Links:
- removed link link3bot
- removed link link3top
- added link link3, mass 0.130; collision box size=0.03 0.04 0.14; visual mesh filename=package://robotic_arm_pkg/meshes/link3.stl scale=0.001 0.001 0.001
- link base: mass None -> 0.170; geometry collision cylinder length=0.035 radius=0.05; visual cylinder length=0.035 radius=0.05
- link gripper_base: mass None -> 0.020
- link link1: mass None -> 0.075; geometry collision cylinder length=0.03 radius=0.035; visual cylinder length=0.03 radius=0.035
- link link2: mass None -> 0.018
- link link4: mass None -> 0.025
Joints:
- removed joint link3bot_link3top
- removed joint link3top_link4
- added joint link3_link4: type revolute, parent link3, child link4, origin xyz=0 0 0.09 rpy=0 0 0, axis 0 1 0, limit lower=-1.57 upper=1.57 effort=1000.0 velocity=0.5
- joint base_link1: origin xyz=0 0 0.035 rpy=0 0 0 -> xyz=0 0 0.0175 rpy=0 0 0
- joint gripper_base_claw_L: origin xyz=0 -0.008 0.018 rpy=0 0 0 -> xyz=0 -0.0125 0.01 rpy=0 0 0
- joint gripper_base_claw_R: origin xyz=0 0.008 0.018 rpy=0 0 0 -> xyz=0 0.0035 0.012 rpy=0 0 0
- joint link1_link2: origin xyz=0 0 0.05 rpy=0 0 0 -> xyz=0 0 0.042 rpy=0 0 0
- joint link2_link3: child link3bot -> link3
- joint link4_gripper_base: origin xyz=-0.01 0 0.055 rpy=0 0 0 -> xyz=-0.01 0 0.06 rpy=0 0 0

Commit message: modified urdf and mesh files

File: robotic_arm_pkg/urdf/arm_meshed.urdf (robot description, URDF)
Before this commit: robot arm_mesh, 9 links, 8 joints
Links:
- link base: mass None -> 0.170
- link gripper_base: mass None -> 0.020
- link link1: mass None -> 0.075
- link link2: mass None -> 0.018
- link link3bot: mass None -> 0.185
- link link3top: mass None -> 0.075
- link link4: mass None -> 0.025

Commit message: added new moveit config package

File: robotic_arm_pkg/urdf/arm_meshed.urdf (robot description, URDF)
Before this commit: robot arm_mesh, 9 links, 8 joints
Links:
- link base: mass 0.170 -> None

Commit message: gazebo integration 6DOF

File: robotic_arm_pkg/urdf/arm_meshed.urdf (robot description, URDF)
Before this commit: robot arm_mesh, 9 links, 8 joints
Links:
- link base: mass None -> 0.170
